File: hardware/comfospot50_full.kicad_pcb (KiCad board)
At the start: 2 copper layers, 86.5 x 27.5 mm, 29 parts, among them U1 ESP32-C3-WROOM-02-H4

Commit message: Add C20252913 connector to hardware design
Parts:
- removed J_PWR_IN1: 24V IN, JCL:CONN-TH_KF239-5.08-2P
- added CN1: 2601-3102, JLC:CONN-TH_4P-P3.5-2601-3102, F.Cu at (140.1, 95.1)

Commit message: Normalize JLC library references
Parts:
- CN1: footprint JLC:CONN-TH_4P-P3.5-2601-3102 -> jlc:CONN-TH_4P-P3.5-2601-3102
Changed lines of the file:
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@@
 		(embedded_fonts no)
 	)
-	(footprint "JLC:CONN-TH_4P-P3.5-2601-3102"
+	(footprint "jlc:CONN-TH_4P-P3.5-2601-3102"
 		(layer "F.Cu")
 		(at 140.075 95.055 90)
@@
 		)
 		(embedded_fonts no)
-		(model "/c/Users/d90509/OneDrive - d-fine GmbH/workspace/comfospot50/hardware/libs/jlc.3dshapes/CONN-TH_4P-P3.5-2601-3102.wrl"
+		(model "${KIPRJMOD}/hardware/libs/jlc.3dshapes/CONN-TH_4P-P3.5-2601-3102.wrl"
 			(offset
 				(xyz 0 0 0)
