File: hardware/comfospot50_full.kicad_sch (KiCad schematic)
At the start: 29 parts, among them U1 ESP32-C3-WROOM-02-H4

Commit message: Add C20252913 connector to hardware design
Parts:
- removed J_PWR_IN1: 24V IN, JCL:CONN-TH_KF239-5.08-2P, symbol JCL:KF239-5.08-2P
- added CN1: 2601-3102, JLC:CONN-TH_4P-P3.5-2601-3102, symbol JLC:2601-3102
- CABLE1, PANEL1: now not fitted
Connections:
- net GND: now also CN1.2
- net at F1.2: now also CN1.1
Changed lines of the file:
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@@
 		(on_board yes)
 		(in_pos_files yes)
-		(dnp no)
+		(dnp yes)
 		(fields_autoplaced yes)
 		(property "Reference" "CABLE1"
@@
 		(on_board yes)
 		(in_pos_files yes)
-		(dnp no)
+		(dnp yes)
 		(fields_autoplaced yes)
 		(property "Reference" "PANEL1"
@@
 	)
 	(symbol
-		(lib_id "JCL:KF239-5.08-2P")
+		(lib_id "JLC:2601-3102")
 		(at 184.15 19.05 90)
 		(unit 1)
@@
 		(dnp no)
 		(fields_autoplaced yes)
-		(property "Reference" "J_PWR_IN1"
+		(property "Reference" "CN1"
 			(at 189.23 16.5099 90)
 			(show_name no)
@@
 			)
 		)
-		(property "Value" "24V IN"
+		(property "Value" "2601-3102"
 			(at 189.23 19.0499 90)
 			(show_name no)
@@
 			)
 		)
-		(property "Footprint" "JCL:CONN-TH_KF239-5.08-2P"
+		(property "Footprint" "JLC:CONN-TH_4P-P3.5-2601-3102"
 			(at 193.04 19.05 0)
 			(hide yes)
@@
 			)
 		)
-		(property "Datasheet" ""
+		(property "Datasheet" "https://www.lcsc.com/datasheet/C20252913.pdf"
 			(at 195.58 19.05 0)
 			(hide yes)
@@
 			)
 		)
-		(property "Manufacturer" "KEFA(科发)"
+		(property "Manufacturer" "WAGO(万可)"
 			(at 198.12 19.05 0)
 			(hide yes)
@@
 			)
 		)
-		(property "MPN" "KF239-5.08-2P"
+		(property "MPN" "2601-3102"
 			(at 200.66 19.05 0)
 			(hide yes)
@@
 			)
 		)
-		(property "LCSC Part" "C976701"
+		(property "LCSC Part" "C20252913"
 			(at 203.2 19.05 0)
 			(hide yes)
@@
 			)
 		)
+		(pin "1"
+		)
 		(pin "2"
-		)
-		(pin "1"
 		)
 		(instances
 			(project "comfospot50_full"
 				(path "/42398dff-893d-443d-90dd-1065dd7a9422"
-					(reference "J_PWR_IN1")
+					(reference "CN1")
 					(unit 1)
 				)

Commit message: Normalize JLC library references
Parts:
- CN1: footprint JLC:CONN-TH_4P-P3.5-2601-3102 -> jlc:CONN-TH_4P-P3.5-2601-3102; symbol JLC:2601-3102 -> jlc:2601-3102
Changed lines of the file:
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@@
 	)
 	(symbol
-		(lib_id "JLC:2601-3102")
+		(lib_id "jlc:2601-3102")
 		(at 184.15 19.05 90)
 		(unit 1)
@@
 			)
 		)
-		(property "Footprint" "JLC:CONN-TH_4P-P3.5-2601-3102"
+		(property "Footprint" "jlc:CONN-TH_4P-P3.5-2601-3102"
 			(at 193.04 19.05 0)
 			(hide yes)

Commit message: Use GitHub component in ESPHome example
Other:
- note added: "led_error"
- note removed: "led_err"
Changed lines of the file:
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@@
 	(generator_version "10.0")
 	(paper "A4")
-	(text "led_filter"
+	(text "led_error"
 		(exclude_from_sim no)
 		(at 48.006 36.83 0)
@@
 		)
 	)
-	(text "led_err"
+	(text "led_filter"
 		(exclude_from_sim no)
-		(at 50.546 185.42 0)
+		(at 52.07 185.42 0)
 		(effects
 			(font
